Commit message: modifications to gpg_remote adding urdf

File: src/gpg_remote/config/gopigo3.urdf (robot description, URDF)
Before this commit: robot gopigo3, 0 links, 0 joints
Links:
- added link base_link
- added link left_wheel_link
- added link right_wheel_link
- added link servo_link
Joints:
- added joint left_wheel: type continuous, parent base_link, child left_wheel_link
- added joint right_wheel: type continuous, parent base_link, child right_wheel_link
- added joint servo: type revolute, parent base_link, child servo_link, limit lower=-3.14 upper=3.14 effort=1000.0 velocity=1000
